File: keyboard/key_matrix.kicad_sch (KiCad schematic)
At the start: 77 parts

Commit message: correct key text
Parts:
- S53: value ` _ -> KP-
Changed lines of the file:
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@@
   (junction (at 101.6 96.52) (diameter 0) (color 0 0 0 0)
   )
-  (junction (at 73.66 83.82) (diameter 0) (color 0 0 0 0)
-  )
   (junction (at 144.78 129.54) (diameter 0) (color 0 0 0 0)
   )
@@
   (junction (at 93.98 129.54) (diameter 0) (color 0 0 0 0)
   )
-  (junction (at 53.34 38.1) (diameter 0) (color 0 0 0 0)
-  )
   (junction (at 91.44 142.24) (diameter 0) (color 0 0 0 0)
   )
@@
     (stroke (width 0) (type default))
   )
-  (wire (pts (xy 73.66 83.82) (xy 73.66 99.06))
-    (stroke (width 0) (type default))
-  )
   (wire (pts (xy 101.6 93.98) (xy 111.76 93.98))
     (stroke (width 0) (type default))
@@
     (stroke (width 0) (type default))
   )
-  (wire (pts (xy 73.66 83.82) (xy 71.12 83.82))
-    (stroke (width 0) (type default))
-  )
   (wire (pts (xy 71.12 111.76) (xy 81.28 111.76))
     (stroke (width 0) (type default))
@@
     (stroke (width 0) (type default))
   )
-  (wire (pts (xy 50.8 29.21) (xy 53.34 29.21))
-    (stroke (width 0) (type default))
-  )
   (wire (pts (xy 60.96 99.06) (xy 63.5 99.06))
     (stroke (width 0) (type default))
@@
     (stroke (width 0) (type default))
   )
-  (wire (pts (xy 73.66 68.58) (xy 73.66 83.82))
+  (wire (pts (xy 73.66 68.58) (xy 73.66 99.06))
     (stroke (width 0) (type default))
   )
@@
   )
   (wire (pts (xy 142.24 144.78) (xy 144.78 144.78))
-    (stroke (width 0) (type default))
-  )
-  (wire (pts (xy 53.34 29.21) (xy 53.34 38.1))
     (stroke (width 0) (type default))
   )
@@
       (effects (font (size 1.27 1.27)))
     )
-    (property "Value" "` _" (at 56.8579 106.68 0)
-      (effects (font (size 1.27 1.27)))
-    )
+    (property "Value" "KP-" (at 56.8579 106.68 0)
+      (effects (font (size 1.27 1.27)))
+    )
