File: keyboard/keyboard.kicad_sch (KiCad schematic)
At the start: 30 parts, among them J1 Keyboard Connector

Commit message: keyboard schematic rev 2
Parts:
- added JP1: KBD7, Jumper:SolderJumper-2_P1.3mm_Bridged_Pad1.0x1.5mm, symbol Jumper:SolderJumper_2_Bridged
- added JP2: LO/RO, Jumper:SolderJumper-2_P1.3mm_Bridged_Pad1.0x1.5mm, symbol Jumper:SolderJumper_2_Bridged
- added R6: ~, Resistor_THT:R_Axial_DIN0309_L9.0mm_D3.2mm_P12.70mm_Horizontal, symbol Device:R_Small_US
Connections:
- net GND: now also JP1.1 (A), JP2.1 (A); no longer E12.1 (Pin_1), E13.1 (Pin_1), J1.3 (Pin_3), Z7.13 (LO/RO)
- net VCC: now also R6.1
- net at E14.1 (Pin_1): now also R6.2
- net KBINH_OUT renamed STROBE
- net ~{SHIFTLOCK} renamed PRINT
- net ~{X15} renamed CLEAR
- new net: E12.1 (Pin_1), JP2.2 (B), Z7.13 (LO/RO)
- new net KBD7: E13.1 (Pin_1), J1.3 (Pin_3), JP1.2 (B)
- no-connect marks 8 -> 7
Other:
- moved on the sheet: C3, C4, C5, C6, C8, D1, E10, E11, E12, E13, E14, E15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
